File: calkabot3d0/schematic/driver.brd (EAGLE design)
At the start: 60.9 x 42.9 mm, 61 parts

Commit message: pcb design
Parts:
- removed BATTERY1, JTAG: (no value), led:CHIPLED_0805
- removed C12: (no value), rcl:C0603
- removed C6, C7, C8: (no value), rcl:CT3528
- removed JP4, JP5: (no value), pinhead:1X02/90
- added I2C_CON, SWD_CON: (no value), pinhead:1X04
- added MA, MB: (no value), pinhead:1X02/90
- added S3: (no value), switch-dil:SD4-01
- C1, C2, C3, C4: value (none) -> 100n
- C5: value (none) -> 100n; device rcl:CT3528 -> rcl:C0603
- I2C, SWD: device pinhead:1X04 -> led:CHIPLED_0805
- moved R19 109.7 mm to (-2.00, 52.0), flipped to the bottom
- moved R17 82.2 mm to (-2.00, 45.0), flipped to the bottom
- moved R18 82.2 mm to (-2.00, 38.0), flipped to the bottom
- moved USB 68.1 mm to (2.71, 12.2), turned to 90 degrees
- moved R2 63.5 mm to (-5.42, 46.3), flipped to the bottom
- moved C17 61.0 mm to (-6.69, 59.0), flipped to the bottom
- moved 12V 60.2 mm to (8.31, 29.9)
- moved C4 58.5 mm to (-7.96, 64.1), flipped to the bottom
- moved C16 57.6 mm to (3.51, 18.4), flipped to the bottom
- moved 3.3V 55.5 mm to (11.7, 30.0)
- moved C19 53.5 mm to (-10.5, 36.2), flipped to the bottom
- moved R1 53.5 mm to (-10.5, 46.3), flipped to the bottom
- moved C3 50.9 mm to (-11.8, 64.1), flipped to the bottom
- moved C15 48.4 mm to (-13.0, 59.0), flipped to the bottom
- moved R3 44.1 mm to (-58.8, 52.7), flipped to the bottom
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Connections:
- new net DIODE: D1.A, S3.1
- new net PB9: R9.2, S2.3, STM32.46
- net BAT+: now also S3.2; no longer D1.A
- net GND: now also C5.2, I2C.C, I2C_CON.3, SWD.C, SWD_CON.4; no longer BATTERY1.C, C12.2, C5.-, C6.-, C7.-, C8.-, I2C.3, JTAG.C, SWD.4
- net N$10: now also SWD.A; no longer JTAG.A
- net N$42: now also MA.2; no longer JP4.2
- net N$43: now also MA.1; no longer JP4.1
- net N$44: now also MB.1; no longer JP5.2
- net N$45: now also MB.2; no longer JP5.1
- net N$9: now also I2C.A; no longer BATTERY1.A
- net PC13: now also R7.2; no longer R9.2, S2.3
- net SCL: now also I2C_CON.2; no longer I2C.2
- net SDA: now also I2C_CON.1; no longer I2C.1
- net SWCLK: now also SWD_CON.3; no longer R7.2, SWD.3
- net SWDA: now also SWD_CON.2; no longer SWD.2
- net VCC_S: now also I2C_CON.4; no longer I2C.4
- net VDD: now also C5.1, SWD_CON.1; no longer C12.1, C5.+, C6.+, C7.+, C8.+, SWD.1
Routing:
- net GND: track 36.9 -> 98.3 mm
- net N$45: track 0.00 -> 16.8 mm
- net N$44: track 0.00 -> 16.6 mm
- net DIODE: track 0.00 -> 15.4 mm
- net N$42: track 0.00 -> 15.0 mm
- net N$43: track 0.00 -> 14.9 mm
- net STAB: track 48.8 -> 59.2 mm
- net BAT+: track 12.5 -> 8.30 mm
- net VDD: track 12.9 -> 8.79 mm, vias 1 -> 0
Other:
- board size 60.9 x 42.9 mm -> 61.9 x 36.8 mm
