File: calkabot3d0/schematic/driver.sch (EAGLE design)
At the start: 61 parts

Commit message: pcb design
Parts:
- removed BATTERY1, JTAG: (no value), led:LEDCHIPLED_0805
- removed C12: (no value), rcl:C-EUC0603
- removed C6, C7, C8: (no value), rcl:CPOL-USCT3528
- added I2C_CON, SWD_CON: (no value), pinhead:PINHD-1X4
- added S3: (no value), switch-dil:SD4-01
- C1, C2, C3, C4: value (none) -> 100n
- C5: value (none) -> 100n; device rcl:CPOL-USCT3528 -> rcl:C-EUC0603
- I2C, SWD: device pinhead:PINHD-1X4 -> led:LEDCHIPLED_0805; SPICEPREFIX (none) -> D
- renumbered JP4 to MA, JP5 to MB
Connections:
- new net DIODE: D1.A, S3.1
- new net PB9: R9.2, S2.3, STM32PORTB_H.PB9
- net BAT+: now also S3.2; no longer D1.A
- net GND: now also C5.2, I2C.C, I2C_CON.3, SWD.C, SWD_CON.4; no longer BATTERY1.C, C12.2, C5.-, C6.-, C7.-, C8.-, I2C.3, JTAG.C, SWD.4
- net N$10: now also SWD.A; no longer JTAG.A
- net N$44: now also MB.1; no longer MB.2
- net N$45: now also MB.2; no longer MB.1
- net N$9: now also I2C.A; no longer BATTERY1.A
- net PC13: now also R7.2; no longer R9.2, S2.3
- net SCL: now also I2C_CON.2; no longer I2C.2
- net SDA: now also I2C_CON.1; no longer I2C.1
- net SWCLK: now also SWD_CON.3; no longer R7.2, SWD.3
- net SWDA: now also SWD_CON.2; no longer SWD.2
- net VCC_S: now also I2C_CON.4; no longer I2C.4
- net VDD: now also C5.1, SWD_CON.1; no longer C12.1, C5.+, C6.+, C7.+, C8.+, SWD.1
Other:
- note added: "sprawdzanie poziomu naładowania baterii"
- moved on the sheet: R17, R18
