File: schematic/driver.sch (EAGLE design)
At the start: 58 parts

Commit message: Add in series stabilisators
Parts:
- removed R13: 65, rcl:R-EU_R0805
- added C6: 100n, rcl:C-EUC0603
- added R20: 150R, rcl:R-EU_R0805
- added R21: 33R, rcl:R-EU_R0805
- BATTERY: value (none) -> WS2812B5050; device led:LEDCHIPLED_0805 -> adafruit:WS2812B5050; SPICEPREFIX D -> (none)
Connections:
- removed net N$8: BATTERY.A, R13.1
- new net DI_LED: R21.2
- new net N$15: BATTERY.VDD, R20.1
- new net N$16: BATTERY.DI, R21.1
- net GND: now also BATTERY.GND, C6.2; no longer BATTERY.C
- net LED2: no longer R13.2
- net STAB: no longer C13.+, LM1117.IN
- net VCC: now also C13.+, J1.VBUS, LM1117.IN, R11.2
- net VDD: now also C6.1, R20.2; no longer J1.VBUS, R11.2
Other:
- moved on the sheet: 12V, 3.3V, C1, C10, C11, C2, C3, C4, C5, C9, I2C, J1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

Commit message: update
Parts:
- removed S1: (no value), switch-dil:SD4-01
- added STM1: STM32F10XCXT6, stm32:STM32F10XCXT6
- added U1: GY-521MPU6050, gy-521:GY-521MPU6050
- S2: device switch-dil:DP03 -> special:SW_DIP-4
Connections:
- removed net TDO: STM32PORTB_L.PB3
- new net INT: STM32PORTB_L.PB3, U1.INT
- net GND: now also STM1RESET.BOOT0, U1.GND; no longer STM32RESET.BOOT0
- net NRST: now also STM1RESET.NRST; no longer STM32RESET.NRST
- net PC13: no longer R7.2
- net SCL: now also U1.SCL
- net SDA: now also U1.SDA
- net SWDIO: now also R7.2
- net VCC: now also S2.5, U1.VCC; no longer S1.2
- net VCC_S: now also S2.4; no longer S1.1
- net VDD: now also S2.7, S2.8; no longer S2.4, S2.5
Other:
- note removed: "Ledy informacyjne"
- moved on the sheet: 3.3V, D1, R3, R8, USB

Commit message: added charger, and over charge protection
Parts:
- removed BATTERY: WS2812B5050, adafruit:WS2812B5050
- removed I2C: (no value), led:LEDCHIPLED_0805
- added C12, C20, C21, C7, C8: 100n, rcl:C-EUC0603
- added D2, D3, D4, D5, D6, D7: S3A, s3x_10:S3A
- added IC1, IC2, IC3: DW01A, DW01A:DW01A
- added LCD1: LPH-7366, lph-7366 (1):LPH-7366
- added R13, R22, R24, R25, R27, R28, R29: 1k, rcl:R-EU_R0805
- added R23, R26: 10k, rcl:R-EU_R0805
- added R30, R31, R32: 100, rcl:R-EU_R0805
- added U$1, U$2, U$3: TP4056, TP4056:TP4056
- R19: value 65 -> 1k
- R20: value 150R -> 10k
- R21: value 33R -> 1k
Connections:
- removed net DI_LED: R21.2
- new net CELL1: R30.2, U$1.BAT
- new net CELL2: R31.2, U$2.BAT
- new net CELL3: R32.2, U$3.BAT
- new net D/C: LCD1.D/C
- new net MOSI: LCD1.SDIN
- new net N$12: D2.C, R13.1
- new net N$13: R19.2, U$1.!CHRG
- new net N$14: D3.C, R19.1
- new net N$18: D4.C, R21.1
- new net N$19: D5.C, R22.1
- new net N$20: R23.2, U$2.PROG
- new net N$21: LCD1.VOUT
- new net N$22: R25.2, U$3.!CHRG
- new net N$23: R24.2, U$3.!STDBY
- new net N$24: D6.C, R24.1
- new net N$25: D7.C, R25.1
- new net N$26: R26.2, U$3.PROG
- new net N$27: C20.1, C21.1, IC2.VCC, IC3.VCC, R30.1, R31.1
- new net N$28: IC3.CS, R29.2
- new net N$29: C12.1, IC1.VCC, R32.1
- new net N$30: IC1.CS, R27.2
- new net N$32: IC2.CS, R28.2
- new net N$8: R22.2, U$2.!CHRG
- new net RES: LCD1./RES
- new net SCE: LCD1./SCE
- new net SCLK: LCD1.SCLK
- net GND: now also C12.2, C20.2, C21.2, C7.2, C8.2, IC1.GND, IC2.GND, IC3.GND, LCD1.GND, R20.1, R23.1, R26.1, R27.1, R28.1, R29.1, U$1.GND, U$1.TEMP, U$2.GND, U$2.TEMP, U$3.GND, U$3.TEMP; no longer BATTERY.GND, I2C.C
- net N$15: now also R20.2, U$1.PROG; no longer BATTERY.VDD, R20.1
- net N$16: now also R21.2, U$2.!STDBY; no longer BATTERY.DI, R21.1
- net N$9: now also R13.2, U$1.!STDBY; no longer I2C.A, R19.1
- net VCC: now also C6.1, C7.1, C8.1, D2.A, D3.A, D4.A, D5.A, D6.A, D7.A, LCD1.OSC, U$1.CE, U$1.VCC, U$2.CE, U$2.VCC, U$3.CE, U$3.VCC
- net VCC_S: no longer R19.2
- net VDD: now also LCD1.VDD; no longer C6.1, R20.2
Other:
- note added: "ładowanie"
- moved on the sheet: C6, R19, R20, R21

Commit message: Added battery managment and motor drivers
Parts:
- removed J2: (no value), SparkFun-Connectors:BATTERY_CONN_DEANS
- removed LM1, LM1117: LM1117MP-3.3, lm1117_11:LM1117MP-3.3
- removed S3: (no value), switch-dil:SD4-01
- removed TB1: POLOLU-713, POLOLU-713:POLOLU-713
- added 7.5K: 7.5k, rcl:R-EU_R0805
- added 7.5K1: 4.5k, rcl:R-EU_R0805
- added D8: CESD5V0D1, Diodes:CESD5V0D1
- added JP1: (no value), pinhead:PINHD-1X3
- added JP2: (no value), pinhead:PINHD-1X2
- added L1, L2: 22uH, rcl:L-USL1812
- added Q2, Q3, Q4: SI1922EDH-T1-GE3, fets:SI1922EDH-T1-GE3
- added R33, R34: 1k, rcl:R-EU_R0805
- added S4: (no value), switch:255SB
- added U$4, U$5: MT3608SOT23-6, MT3608:MT3608SOT23-6
- added U$6, U$7: TB6612FNG, TB6612FNG:TB6612FNG
- C13, C14, C18, C19: value 10u -> 100n; device rcl:CPOL-USCT3528 -> rcl:C-EUC0603
- D1: value S3A -> CESD5V0D1; device s3x_10:S3A -> Diodes:CESD5V0D1
Connections:
- removed net DIODE: D1.A, S3.1
- removed net N$42: MA.2, TB1.BO2
- removed net N$43: MA.1, TB1.BO1
- removed net N$44: MB.1, TB1.AO2
- removed net N$45: MB.2, TB1.AO1
- new net A01: MA.2, U$6.A01, U$6.A01., U$6.B01, U$6.B01.
- new net A02: MB.2, U$7.A01, U$7.A01., U$7.B01, U$7.B01.
- new net AO1: MB.1, U$7.A02, U$7.A02., U$7.B02, U$7.B02.
- new net AO2: MA.1, U$6.A02, U$6.A02., U$6.B02, U$6.B02.
- new net BAT_ON: C13.1, C18.1, L1.1, L2.1, S4.O, U$4.EN, U$4.IN, U$5.EN, U$5.IN, U$6.VM1, U$6.VM2, U$6.VM3, U$7.VM1, U$7.VM2, U$7.VM3
- new net N$28: IC1.OC, Q2G$2.G
- new net N$31: Q2G$1.D, Q2G$2.D
- new net N$33: C20.1, IC2.VCC, R31.1
- new net N$34: IC2.OD, Q3G$1.G
- new net N$35: IC2.OC, Q3G$2.G
- new net N$36: Q3G$1.D, Q3G$2.D
- new net N$38: C21.1, IC3.VCC, R30.1
- new net N$39: IC3.OD, Q4G$1.G
- new net N$40: IC3.OC, Q4G$2.G
- new net N$41: Q4G$1.D, Q4G$2.D
- new net N$47: D1.A, L1.2, U$4.SW
- new net N$49: D8.A, L2.2, U$5.SW
- new net N$50: 7.5K1.1, R33.2, U$5.FB
- new net N$51: 7.5K.1, R34.2, U$4.FB
- new net VBUS: J1.VBUS, JP1.2
- new net VUSB: C6.1, C7.1, C8.1, D2.A, D3.A, D4.A, D5.A, D6.A, D7.A, JP1.3, U$1.CE, U$1.VCC, U$2.CE, U$2.VCC, U$3.CE, U$3.VCC
- net BAT+: now also JP2.2, R17.2, S4.P; no longer J2.+, S3.2
- net GND: now also C13.2, C14.2, C18.2, C19.2, JP2.1, Q2G$1.S, Q2G$2.S, Q3G$1.S, Q3G$2.S, Q4G$1.S, Q4G$2.S, R33.1, R34.1, U$4.GND, U$5.GND, U$6.GND, U$6.PGND1, U$6.PGND1., U$6.PGND2, U$6.PGND2., U$7.GND, U$7.PGND1, U$7.PGND1., U$7.PGND2, U$7.PGND2.; no longer C13.-, C14.-, C18.-, C19.-, J2.-, LM1.GND, LM1117.GND, TB1.GND
- net MA1: now also U$6.AIN1, U$6.BIN1; no longer TB1.AIN1
- net MA2: now also U$6.AIN2, U$6.BIN2; no longer TB1.AIN2
- net MB1: now also U$7.AIN1, U$7.BIN1; no longer TB1.BIN1
- net MB2: now also U$7.AIN2, U$7.BIN2; no longer TB1.BIN2
- net N$27: now also IC1.OD, Q2G$1.G; no longer C20.1, C21.1, IC2.VCC, IC3.VCC, R30.1, R31.1
- net PWMA: now also U$6.PWMA, U$6.PWMB; no longer TB1.PWMA
- net PWMB: now also U$7.PWMA, U$7.PWMB; no longer TB1.PWMB
- net STAB: no longer C18.+, D1.C, LM1.IN, R17.2, TB1.VMOT
- net VCC: now also 7.5K.2, C14.1, D1.C, JP1.1, U$6.STBY, U$6.VCC, U$7.STBY, U$7.VCC; no longer C13.+, C19.+, C6.1, C7.1, C8.1, D2.A, D3.A, D4.A, D5.A, D6.A, D7.A, J1.VBUS, LM1.OUT, LM1117.IN, TB1.!STBY, TB1.VCC, U$1.CE, U$1.VCC, U$2.CE, U$2.VCC, U$3.CE, U$3.VCC
- net VDD: now also 7.5K1.2, C19.1, D8.C; no longer C14.+, LM1117.OUT
Other:
- note added: "Ochrona ogniw"
- note added: "przetwornice"
- note removed: "Zasilanie'"
- moved on the sheet: C12, C20, C21, C6, C7, C8, D2, D3, D4, D5, D6, D7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

Commit message: added MPU6050 to board, and two motor drivers
Parts:
- removed U1: GY-521MPU6050, gy-521:GY-521MPU6050
- added C22, C23, C25, C27, C29, C31, C32: 100n, rcl:C-EUC0603
- added C24: 2.2n, rcl:C-EUC0603
- added C26: 10nF, rcl:C-EUC0603
- added C28, C30: 10uF, rcl:C-EUC0603
- added IC4: MPU6050, invensense:MPU6050
Connections:
- new net N$42: C22.1, IC4G$1.REGOUT
- new net N$43: C23.1
- new net N$44: IC4G$1.FSYNC
- new net N$45: C24.1, IC4G$1.CPOUT
- new net N$48: C27.1, C28.1, U$6.VM1
- net BAT_ON: now also C29.1, C30.1; no longer U$6.VM1
- net GND: now also C22.2, C23.2, C24.2, C25.2, C26.2, C27.2, C28.2, C29.2, C30.2, C31.2, C32.2, IC4G$1.CLKIN, IC4G$1.GND, IC4G$1.GND@1; no longer U1.GND
- net INT: now also IC4G$1.INT; no longer U1.INT
- net SCL: now also IC4G$1.SCL; no longer U1.SCL
- net SDA: now also IC4G$1.SDA; no longer U1.SDA
- net VCC: now also C31.1, C32.1; no longer U1.VCC
- net VDD: now also C25.1, C26.1, IC4G$1.VDD, IC4G$1.VLOGIC
Other:
- note added: "Akcelerator"
- moved on the sheet: 7.5K, 7.5K1, C12, C13, C14, C18, C19, C20, C21, C6, C7, C8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

Commit message: 0
Parts:
- removed 12V: (no value), led:LEDCHIPLED_0805
- removed R4: 500, rcl:R-EU_R0805
- removed STM1: STM32F10XCXT6, stm32:STM32F10XCXT6
- added 3.3V1, 3.3V2, 3.3V3: (no value), led:LEDCHIPLED_0805
Connections:
- removed net STAB: R4.2
- new net N$1: C15.1, STM32AN_POWER.VBAT
- new net N$5: RESET.3
- new net N$52: 3.3V2.C, R6.2
- new net N$53: 3.3V3.C, R5.2
- new net N$59: C31.1, U$6.STBY
- new net N$60: C32.1, U$7.STBY
- net GND: no longer 12V.C, RESET.3, STM1RESET.BOOT0
- net N$2: now also 3.3V1.C, R9.2; no longer 12V.A, R4.1
- net NRST: no longer STM1RESET.NRST
- net PB9: now also 3.3V1.A; no longer R9.2
- net PC14: now also 3.3V2.A; no longer R6.2
- net PC15: now also 3.3V3.A; no longer R5.2
- net VCC: no longer C31.1, C32.1, U$6.STBY, U$7.STBY
- net VDD: no longer C15.1, STM32AN_POWER.VBAT
Other:
- moved on the sheet: 3.3V, 7.5K, 7.5K1, C1, C10, C11, C12, C13, C14, C15, C16, C17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

Commit message: SD Card added
Parts:
- removed C3: 100n, rcl:C-EUC0603
- added JP4: (no value), pinhead:PINHD-2X3
- added R35: 50, rcl:R-EU_R0805
- added R37, R38, R39, R4: 50k, rcl:R-EU_R0805
- added SD_CARD: (no value), Wurth_Elektronik_Electromechanic_Input-Output_Connectors_rev16a:693071010811
Connections:
- removed net N$1: C15.1, STM32AN_POWER.VBAT
- removed net N$59: C31.1, U$6.STBY
- removed net N$60: C32.1, U$7.STBY
- removed net S1: STM32PORTA_L.PA7
- removed net S2: STM32PORTA_L.PA6
- removed net S3: STM32PORTA_L.PA5
- removed net S4: STM32PORTA_L.PA4
- new net BOOT0: JP4.4, STM32RESET.BOOT0
- new net BOOT1: JP4.3, STM32PORTB_L.PB2
- new net CS: R4.1, SD_CARD.CD/DAT3, STM32PORTA_L.PA4
- new net MISO: R38.1, SD_CARD.DAT0, STM32PORTA_L.PA6
- new net N$61: R35.1, SD_CARD.DAT2
- new net N$63: R39.1, SD_CARD.DAT1
- new net SCK: SD_CARD.CLK, STM32PORTA_L.PA5
- new net SCL1: STM32PORTB_L.PB6
- new net SCL2: STM32PORTB_H.PB10
- new net SDA1: STM32PORTB_L.PB7
- new net SDA2: STM32PORTB_H.PB11
- new net VSS: STM32AN_POWER.VSSA
- net GND: now also JP4.5, JP4.6, SD_CARD.VSS; no longer C3.2, STM32AN_POWER.VSSA, STM32PORTB_L.PB2
- net MA2: now also STM32PORTB_H.PB9; no longer STM32PORTB_H.PB11
- net MB1: now also STM32PORTB_H.PB14; no longer STM32PORTB_H.PB13
- net MB2: now also STM32PORTB_H.PB13; no longer STM32PORTB_H.PB14
- net MOSI: now also R37.1, SD_CARD.CMD, STM32PORTA_L.PA7
- net NRST: now also STM32RESET.NRST
- net PB9: no longer STM32PORTB_H.PB9
- net PWMA: now also STM32PORTB_H.PB8; no longer STM32PORTB_H.PB10
- net SCL: no longer STM32PORTB_L.PB6
- net SDA: no longer STM32PORTB_L.PB7
- net VCC: now also C31.1, C32.1, U$6.STBY, U$7.STBY
- net VDD: now also C15.1, JP4.1, JP4.2, R35.2, R37.2, R38.2, R39.2, R4.2, SD_CARD.VDD, STM32AN_POWER.VBAT; no longer C3.1
Other:
- note removed: "Akcelerator"
- moved on the sheet: C1, C10, C11, C15, C16, C2, C4, C5, Q1, STM32AN_POWER, STM32PORTA_H, STM32PORTA_L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

Commit message: Added piheads for sensors. Added transoptors.
Parts:
- added JP10, JP3, JP5, JP6, JP7, JP8, JP9: (no value), pinhead:PINHD-1X4
- added R36, R41, R43, R45: 20k, rcl:R-EU_R0805
- added R40, R42, R44, R46: 200, rcl:R-EU_R0805
- added U$10, U$11, U$8, U$9: CNY70, cny70:CNY70
- R35: value 50 -> 50k
Connections:
- removed net LED2: STM32PORTA_L.PA2
- removed net N$17: STM32PORTA_H.PA8
- removed net PB9: 3.3V1.A, S2.3
- removed net PC13: STM32PORTC.PC13
- removed net PC14: 3.3V2.A, S2.2, STM32PORTC.PC14
- removed net S0: STM32PORTB_L.PB0
- removed net TRST: STM32PORTB_L.PB4
- new net ADC1: R36.1, STM32PORTA_L.PA1, U$8.COL
- new net ADC2: R41.1, STM32PORTA_L.PA2, U$9.COL
- new net ADC3: R43.1, STM32PORTA_L.PA3, U$10.COL
- new net ADC4: R45.1, U$11.COL
- new net N$1: R40.1, U$8.A
- new net N$56: R42.1, U$9.A
- new net N$57: STM32PORTB_L.PB5
- new net N$62: R44.1, U$10.A
- new net N$65: R43.2, R44.2
- new net N$66: R46.1, U$11.A
- new net N$68: R45.2, R46.2
- new net SW1: 3.3V3.A, S2.1, STM32PORTA_H.PA8
- new net SW2: 3.3V2.A, S2.2, STM32PORTA_H.PA9
- new net SW3: 3.3V1.A, S2.3, STM32PORTA_H.PA10
- net BAT: now also STM32PORTA_L.PA0; no longer STM32PORTA_L.PA3
- net BUT: now also STM32PORTB_L.PB0, STM32PORTC.PC14; no longer STM32PORTB_L.PB1
- net GND: now also JP10.2, JP3.2, JP5.2, JP6.2, JP7.2, JP8.2, JP9.2, U$10.C, U$10.EMI, U$11.C, U$11.EMI, U$8.C, U$8.EMI, U$9.C, U$9.EMI
- net INT: now also STM32PORTB_L.PB1; no longer STM32PORTB_L.PB3
- net LED1: now also STM32PORTB_L.PB3, STM32PORTB_L.PB4, STM32PORTC.PC13; no longer STM32PORTA_L.PA1
- net PC15: no longer 3.3V3.A, S2.1
- net SCL2: now also JP10.3, JP3.3, JP5.3, JP6.3, JP7.3, JP8.3, JP9.3
- net SDA2: now also JP10.4, JP3.4, JP5.4, JP6.4, JP7.4, JP8.4, JP9.4
- net VCC: now also JP10.1, JP3.1, JP5.1, JP6.1, JP7.1, JP8.1, JP9.1, R36.2, R40.2, R41.2, R42.2
